File: hardware/SilentStepStick-TMC2130_v10.brd (EAGLE design)
At the start: 15.2 x 20.3 mm, 26 parts, among them IC1 TMC2100-LA, X1 PASSER-07, X2 PASSER-07

Commit message: updated schematics
Parts:
- IC1: value TMC2100-LA -> TMC2130-LA
Changed lines of the file:
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@@
 <?xml version="1.0" encoding="utf-8"?>
 <!DOCTYPE eagle SYSTEM "eagle.dtd">
-<eagle version="7.5.0">
+<eagle version="7.6.0">
 <drawing>
 <settings>
@@
 <setting verticaltext="up"/>
 </settings>
-<grid distance="0.635" unitdist="mm" unit="mm" style="lines" multiple="1" display="yes" altdistance="0.0025" altunitdist="inch" altunit="inch"/>
+<grid distance="0.05" unitdist="inch" unit="inch" style="lines" multiple="1" display="yes" altdistance="0.025" altunitdist="inch" altunit="inch"/>
 <layers>
 <layer number="1" name="Top" color="4" fill="1" visible="yes" active="yes"/>
@@
 <attribute name="NAME" x="12.1285" y="10.9855" size="0.4064" layer="25" font="vector" ratio="10" align="center"/>
 </element>
-<element name="IC1" library="we-chip" package="QFN36-PAD" value="TMC2100-LA" x="7.004" y="12" smashed="yes">
+<element name="IC1" library="we-chip" package="QFN36-PAD" value="TMC2130-LA" x="7.004" y="12" smashed="yes">
 <attribute name="NAME" x="4.5275" y="14.8575" size="0.4064" layer="25" font="vector" ratio="10" align="center"/>
 </element>
