File: hardware/SilentStepStick_v12_5V.sch (EAGLE design)
At the start: 30 parts, among them IC1 TMC2100-LA, X1 PASSER-07, X2 PASSER-07

Commit message: updated schematics
Parts:
- IC1: device we-chip:TMC2100-LA -> we-chip:TMC21X0-LA
Changed lines of the file:
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@@
 <?xml version="1.0" encoding="utf-8"?>
 <!DOCTYPE eagle SYSTEM "eagle.dtd">
-<eagle version="7.5.0">
+<eagle version="7.6.0">
 <drawing>
 <settings>
@@
 <setting verticaltext="up"/>
 </settings>
-<grid distance="0.05" unitdist="inch" unit="inch" style="lines" multiple="1" display="yes" altdistance="0.025" altunitdist="inch" altunit="inch"/>
+<grid distance="0.1" unitdist="inch" unit="inch" style="lines" multiple="1" display="no" altdistance="0.01" altunitdist="inch" altunit="inch"/>
 <layers>
 <layer number="1" name="Top" color="4" fill="1" visible="no" active="no"/>
@@
 <part name="R5" library="we-rcl" deviceset="RESISTOR" device="-0402" value="20k"/>
 <part name="R1" library="we-rcl" deviceset="RESISTOR" device="-0402" value="10"/>
-<part name="IC1" library="we-chip" deviceset="TMC2100" device="-LA"/>
+<part name="IC1" library="we-chip" deviceset="TMC21X0" device="-LA" value="TMC2100-LA"/>
 <part name="GND17" library="supply1" deviceset="GND" device=""/>
 <part name="P+3" library="supply1" deviceset="+5V" device=""/>
